File: CO2/CO2.sch (KiCad schematic (older format))
At the start: 29 parts, among them J1 Conn_Coaxial, J2 Display, J3 SCD30, J4 JST, J5 Conn_Coaxial, Q1 Q_NPN_BCE, U1 NodeMCU1.0(ESP-12E), U2 RFM95W-868S2, U3 MAX-8Q, U4 MCP73831-2-OT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

Commit message: first draft
Parts:
- JP1: symbol Device:Jumper_NC_Small -> CO2-rescue:Jumper_NC_Small-Device
- U1: symbol ESP8266:NodeMCU_1.0_(ESP-12E) -> CO2-rescue:NodeMCU_1.0_(ESP-12E)-ESP8266
- U5: symbol Regulator_Linear:AP2112K-3.3 -> CO2-rescue:AP2112K-3.3-Regulator_Linear
Changed lines of the file:
@@
 $EndComp
 $Comp
-L ESP8266:NodeMCU_1.0_(ESP-12E) U1
+L CO2-rescue:NodeMCU_1.0_(ESP-12E)-ESP8266 U1
 U 1 1 5B936524
 P 8100 2000
@@
 NoConn ~ 7300 1700
 $Comp
-L Regulator_Linear:AP2112K-3.3 U5
+L CO2-rescue:AP2112K-3.3-Regulator_Linear U5
 U 1 1 5F77DDDD
 P 4375 6600
@@
 	10200 3575 10050 3575
 $Comp
-L Device:Jumper_NC_Small JP1
+L CO2-rescue:Jumper_NC_Small-Device JP1
 U 1 1 5F84B155
 P 2250 1750
