File: CO2/CO2.kicad_pcb (KiCad board)
At the start: 2 copper layers, 26.7 x 48.9 mm, 29 parts, among them J1 Conn_Coaxial, J2 Display, J3 SCD30, J4 JST, J5 Conn_Coaxial, Q1 Q_NPN_BCE, U1 NodeMCU1.0(ESP-12E), U2 RFM95W-868S2, U3 MAX-8Q, U4 MCP73831-2-OT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

Commit message: first draft
Parts:
- removed J2: Display, Connector_PinHeader_2.54mm:PinHeader_1x04_P2.54mm_Vertical
- moved R2 2.54 mm to (134.6, 139.1)
- moved R3 2.54 mm to (137.2, 139.1)
- turned C1 to 90 degrees
- turned C5 to 90 degrees
- turned R4 to 90 degrees
- turned U4 to 0 degrees
Routing:
- net +3V3: track 14.1 -> 58.4 mm, vias 0 -> 2
- net LED: track 6.61 -> 40.7 mm, vias 0 -> 1
- net A0: track 2.50 -> 36.0 mm
- net RST: track 0.00 -> 17.6 mm, vias 0 -> 1
- net RXD: track 0.00 -> 12.9 mm
- net GND: track 0.00 -> 11.8 mm
- net CLK: track 19.4 -> 29.3 mm
- net +BATT: track 22.2 -> 17.7 mm
- net IRQ: track 22.7 -> 18.7 mm
- net +5V: track 55.0 -> 51.2 mm
- net CIPO: track 24.4 -> 27.8 mm
- net COPI: track 28.2 -> 31.2 mm
- net Net-(R1-Pad2): track 5.76 -> 4.15 mm
- net SCL: track 33.7 -> 34.8 mm
- net CS: track 24.5 -> 25.6 mm
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Other:
- board text added: "5V"
- board text added: "G"
- board text added: "SCL"
- board text added: "SDA"

Commit message: final board
Routing:
- net GND: track 11.8 -> 5.14 mm, vias 0 -> 23
- net CLK: track 29.3 -> 30.0 mm
