File: CO2/CO2.kicad_pcb (KiCad board)
At the start: 2 copper layers, 26.7 x 48.9 mm, 28 parts, among them J1 Conn_Coaxial, J3 SCD30, J4 JST, J5 Conn_Coaxial, Q1 Q_NPN_BCE, U1 NodeMCU, U2 RFM95W-868S2, U3 MAX-8Q, U4 MCP73831, U5 AP2112K

Commit message: add BME680
Parts:
- removed J3: SCD30, Connector_PinHeader_2.54mm:PinHeader_1x06_P2.54mm_Vertical
- added C6: 100n, Capacitor_SMD:C_0603_1608Metric, F.Cu at (135.9, 105.4)
- added C7: 100n, Capacitor_SMD:C_0603_1608Metric, F.Cu at (129.5, 105.4)
- added J2: Display, Connector_PinHeader_2.54mm:PinHeader_1x04_P2.54mm_Vertical, F.Cu at (141.4, 139.7)
- added U6: BME680, Package_LGA:Bosch_LGA-8_3x3mm_P0.8mm_ClockwisePinNumbering, F.Cu at (132.7, 105.4)
- U1: value NodeMCU -> NodeMCU1.0(ESP-12E)
- U4: value MCP73831 -> MCP73831-2-OT
- U5: value AP2112K -> AP2112K-3.3
Routing:
- net +3V3: track 58.4 -> 73.5 mm, vias 2 -> 3
- net SCL: track 34.8 -> 43.1 mm
- net SDA: track 35.0 -> 40.2 mm
- net RST: track 17.6 -> 20.4 mm, vias 1 -> 2
- net GND: track 5.14 -> 7.28 mm
- added copper zone on F.Cu, net +3V3
Other:
- rule solder_mask_min_width: 0.25 -> 0.125
- board text added: "www.hacKNology.de @ttn_kn"

Commit message: do not use this design
Connections:
- U3 pad 14: (no net) -> Net-(R8-Pad1)
Other:
- board text added: "DO NOT USE THIS DESIGN !"
Changed lines of the file:
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@@
   (general
     (thickness 1.55)
-    (drawings 17)
+    (drawings 18)
     (tracks 230)
     (zones 0)
     (modules 31)
-    (nets 27)
+    (nets 28)
   )
   (page A4)
@@
   (net 25 "Net-(J5-Pad1)")
   (net 26 "Net-(R7-Pad1)")
+  (net 27 "Net-(R8-Pad1)")
   (net_class Default "This is the default net class."
     (clearance 0.2)
@@
     (add_net "Net-(D1-Pad4)")
     (add_net "Net-(D2-Pad2)")
-    (add_net "Net-(D3-Pad2)")
     (add_net "Net-(D4-Pad1)")
     (add_net "Net-(D5-Pad2)")
@@
     (add_net "Net-(R4-Pad1)")
     (add_net "Net-(R7-Pad1)")
-    (add_net "Net-(U1-Pad12)")
-    (add_net "Net-(U1-Pad13)")
-    (add_net "Net-(U1-Pad2)")
-    (add_net "Net-(U1-Pad3)")
-    (add_net "Net-(U1-Pad4)")
-    (add_net "Net-(U1-Pad5)")
-    (add_net "Net-(U1-Pad6)")
-    (add_net "Net-(U1-Pad7)")
-    (add_net "Net-(U1-Pad8)")
-    (add_net "Net-(U1-Pad9)")
-    (add_net "Net-(U2-Pad11)")
-    (add_net "Net-(U2-Pad12)")
-    (add_net "Net-(U2-Pad15)")
-    (add_net "Net-(U2-Pad16)")
-    (add_net "Net-(U2-Pad7)")
-    (add_net "Net-(U3-Pad13)")
-    (add_net "Net-(U3-Pad14)")
-    (add_net "Net-(U3-Pad15)")
-    (add_net "Net-(U3-Pad16)")
-    (add_net "Net-(U3-Pad17)")
-    (add_net "Net-(U3-Pad18)")
-    (add_net "Net-(U3-Pad3)")
-    (add_net "Net-(U3-Pad5)")
-    (add_net "Net-(U3-Pad9)")
-    (add_net "Net-(U5-Pad4)")
+    (add_net "Net-(R8-Pad1)")
     (add_net RST)
     (add_net RXD)
     (add_net SCL)
     (add_net SDA)
-    (add_net TXD)
   )
   (module Package_LGA:Bosch_LGA-8_3x3mm_P0.8mm_ClockwisePinNumbering (layer F.Cu)
@@
     (pad 16 smd roundrect (at 4.75 2.2 270) (size 1.8 0.8) (layers B.Cu B.Paste B.Mask) (roundrect_rratio 0.25))
     (pad 15 smd roundrect (at 4.75 1.1 270) (size 1.8 0.8) (layers B.Cu B.Paste B.Mask) (roundrect_rratio 0.25))
-    (pad 14 smd roundrect (at 4.75 0 270) (size 1.8 0.8) (layers B.Cu B.Paste B.Mask) (roundrect_rratio 0.25))
+    (pad 14 smd roundrect (at 4.75 0 270) (size 1.8 0.8) (layers B.Cu B.Paste B.Mask) (roundrect_rratio 0.25)
+      (net 27 "Net-(R8-Pad1)"))
     (pad 13 smd roundrect (at 4.75 -1.1 270) (size 1.8 0.8) (layers B.Cu B.Paste B.Mask) (roundrect_rratio 0.25))
     (pad 12 smd roundrect (at 4.75 -2.2 270) (size 1.8 0.8) (layers B.Cu B.Paste B.Mask) (roundrect_rratio 0.25)
@@
     )
   )
+  (gr_text "DO NOT USE THIS DESIGN !" (at 130.81 102.235 45) (layer Cmts.User)
+    (effects (font (size 12 12) (thickness 2)))
+  )
   (gr_text "www.hacKNology.de\n@ttn_kn" (at 126.365 120.65 90) (layer F.SilkS)
