File: PIS/PIS.kicad_pcb (KiCad board)
At the start: 2 copper layers, 26.7 x 48.9 mm, 24 parts, among them J1 Capacitive Sensor, J2 Conn_01x03, J3 Serial, J4 Screw_Terminal_01x04, J5 Resistive Sensor, K1 G5V-1, Q1 BC547, Q3 BC547, U1 NodeMCU1.0(ESP-12E), U2 TSOP17xx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

Commit message: kicad-exports and CO2 module
Parts:
- JP1: value Jumper_2_Open -> NO
Changed lines of the file:
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@@
-(kicad_pcb (version 20171130) (host pcbnew 5.1.5-52549c5~86~ubuntu18.04.1)
+(kicad_pcb (version 20171130) (host pcbnew 5.1.5+dfsg1-2build2)
   (general
     (thickness 1.55)
-    (drawings 24)
+    (drawings 22)
     (tracks 57)
     (zones 0)
@@
   (title_block
     (title NodeMCU_PIS)
-    (date 2020-03-29)
+    (date 2020-10-04)
     (company https://nerdyscout.github.io/NodeMCU/PIS)
   )
   (layers
-    (0 F.Cu mixed)
-    (31 B.Cu mixed)
-    (32 B.Adhes user)
-    (33 F.Adhes user)
-    (34 B.Paste user)
-    (35 F.Paste user)
-    (36 B.SilkS user)
-    (37 F.SilkS user)
+    (0 F.Cu mixed hide)
+    (31 B.Cu mixed hide)
+    (32 B.Adhes user hide)
+    (33 F.Adhes user hide)
+    (34 B.Paste user hide)
+    (35 F.Paste user hide)
+    (36 B.SilkS user hide)
+    (37 F.SilkS user hide)
     (38 B.Mask user)
-    (39 F.Mask user)
+    (39 F.Mask user hide)
     (40 Dwgs.User user)
     (41 Cmts.User user)
@@
     (46 B.CrtYd user)
     (47 F.CrtYd user)
-    (48 B.Fab user hide)
-    (49 F.Fab user hide)
+    (48 B.Fab user)
+    (49 F.Fab user)
   )
   (setup
@@
       (effects (font (size 1 1) (thickness 0.15)))
     )
-    (fp_text value Jumper_2_Open (at 0 1.9 90) (layer F.Fab)
+    (fp_text value NO (at 0 0 90) (layer F.Fab)
       (effects (font (size 1 1) (thickness 0.15)))
     )
@@
       (effects (font (size 1 1) (thickness 0.15)))
     )
-    (fp_text value "Resistive Sensor" (at 0 9.95 270) (layer F.Fab)
+    (fp_text value "Resistive Sensor" (at 0 3.81) (layer F.Fab) hide
       (effects (font (size 1 1) (thickness 0.15)))
     )
@@
       (effects (font (size 1 1) (thickness 0.15)))
     )
-    (fp_text value CS (at 6.35 0) (layer F.Fab)
+    (fp_text value CS (at 6.35 0) (layer F.Fab) hide
       (effects (font (size 1 1) (thickness 0.15)))
     )
@@
       (effects (font (size 1 1) (thickness 0.15)))
     )
-    (fp_text value MOSI (at 6.35 0) (layer F.Fab)
+    (fp_text value MOSI (at 6.35 0) (layer F.Fab) hide
       (effects (font (size 1 1) (thickness 0.15)))
     )
@@
       (effects (font (size 1 1) (thickness 0.15)))
     )
-    (fp_text value MISO (at 6.35 0) (layer F.Fab)
+    (fp_text value MISO (at 6.35 0) (layer F.Fab) hide
       (effects (font (size 1 1) (thickness 0.15)))
     )
@@
       (effects (font (size 1 1) (thickness 0.15)))
     )
-    (fp_text value CLK (at 6.35 0) (layer F.Fab)
+    (fp_text value CLK (at 6.35 0) (layer F.Fab) hide
       (effects (font (size 1 1) (thickness 0.15)))
     )
@@
       (effects (font (size 1 1) (thickness 0.15)))
     )
-    (fp_text value BC547 (at 1.27 1.905 180) (layer F.Fab)
+    (fp_text value BC547 (at 1.27 0 180) (layer F.Fab)
       (effects (font (size 1 1) (thickness 0.15)))
     )
@@
     (fp_line (start -0.5 1.75) (end 3 1.75) (layer F.Fab) (width 0.1))
     (fp_line (start -0.53 1.85) (end 3.07 1.85) (layer F.SilkS) (width 0.12))
-    (fp_text user %R (at 3.175 -2.54 270) (layer F.Fab)
+    (fp_text user %R (at 1.27 -1.27) (layer F.Fab)
       (effects (font (size 1 1) (thickness 0.15)))
     )
@@
       (effects (font (size 1 1) (thickness 0.15)))
     )
-    (fp_text value 1N4148 (at 3.81 2.12 270) (layer F.Fab)
+    (fp_text value 1N4148 (at 3.81 -1.905 270) (layer F.Fab)
       (effects (font (size 1 1) (thickness 0.15)))
     )
@@
       (effects (font (size 1 1) (thickness 0.15)))
     )
-    (fp_text user K (at 0 -1.8 270) (layer F.Fab)
+    (fp_text user K (at 0 -1.905 270) (layer F.Fab) hide
       (effects (font (size 1 1) (thickness 0.15)))
     )
@@
       (effects (font (size 1 1) (thickness 0.15)))
     )
-    (fp_text value G5V-1 (at 1.905 6.35 180) (layer F.Fab)
-      (effects (font (size 1 1) (thickness 0.15)))
-    )
-    (fp_text user %R (at 3.175 6.35 180) (layer F.Fab)
+    (fp_text value G5V-1 (at 1.905 1.27 180) (layer F.Fab)
+      (effects (font (size 1 1) (thickness 0.15)))
+    )
+    (fp_text user %R (at 3.175 1.27 180) (layer F.Fab)
       (effects (font (size 1 1) (thickness 0.15)))
     )
@@
       (effects (font (size 1 1) (thickness 0.15)))
     )
-    (fp_text value BC547 (at 1.27 1.905) (layer F.Fab)
+    (fp_text value BC547 (at 1.27 0) (layer F.Fab)
       (effects (font (size 1 1) (thickness 0.15)))
     )
@@
     (fp_line (start -0.5 1.75) (end 3 1.75) (layer F.Fab) (width 0.1))
     (fp_line (start -0.53 1.85) (end 3.07 1.85) (layer F.SilkS) (width 0.12))
-    (fp_text user %R (at 3.175 -2.54 270) (layer F.Fab)
+    (fp_text user %R (at 1.27 -1.27) (layer F.Fab)
       (effects (font (size 1 1) (thickness 0.15)))
     )
@@
       (effects (font (size 1 1) (thickness 0.15)) (justify mirror))
     )
-    (fp_text value "NodeMCU1.0(ESP-12E)" (at 12.065 0) (layer B.Fab)
+    (fp_text value "NodeMCU1.0(ESP-12E)" (at 10.16 -2.54) (layer B.Fab)
       (effects (font (size 1 1) (thickness 0.15)) (justify mirror))
     )
     (fp_line (start -0.127 6.096) (end -1.143 5.08) (layer B.Fab) (width 0.1))
-    (fp_text user %R (at 11.43 1.905) (layer B.Fab)
+    (fp_text user %R (at 10.16 -1.27) (layer B.Fab)
       (effects (font (size 1 1) (thickness 0.15)) (justify mirror))
     )
@@
     (effects (font (size 1 1) (thickness 0.15)))
   )
-  (dimension 26.67 (width 0.15) (layer Dwgs.User)
-    (gr_text "26,670 mm" (at 132.715 95.22) (layer Dwgs.User)
-      (effects (font (size 1 1) (thickness 0.15)))
-    )
-    (feature1 (pts (xy 146.05 104.14) (xy 146.05 95.933579)))
-    (feature2 (pts (xy 119.38 104.14) (xy 119.38 95.933579)))
-    (crossbar (pts (xy 119.38 96.52) (xy 146.05 96.52)))
-    (arrow1a (pts (xy 146.05 96.52) (xy 144.923496 97.106421)))
-    (arrow1b (pts (xy 146.05 96.52) (xy 144.923496 95.933579)))
-    (arrow2a (pts (xy 119.38 96.52) (xy 120.506504 97.106421)))
-    (arrow2b (pts (xy 119.38 96.52) (xy 120.506504 95.933579)))
-  )
-  (dimension 48.89011 (width 0.15) (layer Dwgs.User)
-    (gr_text "48,890 mm" (at 154.335 127.319945 270) (layer Dwgs.User)
-      (effects (font (size 1 1) (thickness 0.15)))
-    )
-    (feature1 (pts (xy 144.78 151.765) (xy 153.621421 151.765)))
-    (feature2 (pts (xy 144.78 102.87489) (xy 153.621421 102.87489)))
-    (crossbar (pts (xy 153.035 102.87489) (xy 153.035 151.765)))
-    (arrow1a (pts (xy 153.035 151.765) (xy 152.448579 150.638496)))
-    (arrow1b (pts (xy 153.035 151.765) (xy 153.621421 150.638496)))
-    (arrow2a (pts (xy 153.035 102.87489) (xy 152.448579 104.001394)))
-    (arrow2b (pts (xy 153.035 102.87489) (xy 153.621421 104.001394)))
-  )
   (gr_text 02.02.2019 (at 130.81 144.145 180) (layer B.SilkS)
