File: PIS/PIS.sch (KiCad schematic (older format))
At the start: 24 parts, among them J1 Capacitive Sensor, J2 Conn_01x03, J3 Serial, J4 Screw_Terminal_01x04, J5 Resistive Sensor, K1 G5V-1, Q1 BC547, Q3 BC547, U1 NodeMCU1.0(ESP-12E), U2 TSOP17xx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

Commit message: upgrade
Parts:
- U1: symbol ESP8266:NodeMCU1.0(ESP-12E) -> PIS-rescue:NodeMCU1.0(ESP-12E)-ESP8266
Changed lines of the file:
@@
 $EndComp
 $Comp
-L ESP8266:NodeMCU1.0(ESP-12E) U1
+L PIS-rescue:NodeMCU1.0(ESP-12E)-ESP8266 U1
 U 1 1 5B936524
 P 8100 2000

Commit message: docu
Other:
- note added: "MQTT"
- note added: "PLANT"
- note added: "use to detect \nwater level"
- note removed: "Alternativ zum Relay!"
- moved on the sheet: JP1, U2
Changed lines of the file:
@@
 P 5700 4800
 F 0 "J4" H 5700 4500 50  0000 C CNN
-F 1 "Screw_Terminal_01x04" V 5850 4800 50  0000 C CNN
+F 1 "Screw_Terminal_01x04" V 5850 4800 50  0001 C CNN
 F 2 "TerminalBlock_TE-Connectivity:TerminalBlock_TE_282834-4_1x04_P2.54mm_Horizontal" H 5700 4800 50  0001 C CNN
 F 3 "~" H 5700 4800 50  0001 C CNN
@@
 	1    0    0    1
 $EndComp
-Wire Wire Line
-	2900 5500 3000 5500
 Wire Wire Line
 	3400 4100 3400 4300
@@
 Wire Wire Line
 	9050 1700 8900 1700
-Text Notes 9500 1300 0    50   ~ 0
+Text Notes 9500 1325 0    50   ~ 0
 LED NodeMCU
-Text Notes 9500 1700 0    50   ~ 0
+Text Notes 9500 1725 0    50   ~ 0
 LED ESP12
 Wire Wire Line
@@
 L Interface_Optical:TSOP17xx U2
 U 1 1 5C55B23F
-P 5800 6750
-F 0 "U2" H 5788 7175 50  0000 C CNN
-F 1 "TSOP17xx" H 5788 7084 50  0000 C CNN
-F 2 "OptoDevice:Vishay_CAST-3Pin" H 5750 6375 50  0001 C CNN
-F 3 "http://www.micropik.com/PDF/tsop17xx.pdf" H 6450 7050 50  0001 C CNN
-F 4 "IR" H 5800 6750 50  0001 C CNN "Variant"
-	1    5800 6750
+P 5800 7000
+F 0 "U2" H 5788 7425 50  0000 C CNN
+F 1 "TSOP17xx" H 5788 7334 50  0000 C CNN
+F 2 "OptoDevice:Vishay_CAST-3Pin" H 5750 6625 50  0001 C CNN
+F 3 "http://www.micropik.com/PDF/tsop17xx.pdf" H 6450 7300 50  0001 C CNN
+F 4 "IR" H 5800 7000 50  0001 C CNN "Variant"
+	1    5800 7000
 	-1   0    0    -1
 $EndComp
@@
 L power:GND #PWR0109
 U 1 1 5C55C2F2
-P 5350 7200
-F 0 "#PWR0109" H 5350 6950 50  0001 C CNN
-F 1 "GND" H 5355 7027 50  0000 C CNN
-F 2 "" H 5350 7200 50  0001 C CNN
-F 3 "" H 5350 7200 50  0001 C CNN
-	1    5350 7200
+P 5350 7450
+F 0 "#PWR0109" H 5350 7200 50  0001 C CNN
+F 1 "GND" H 5355 7277 50  0000 C CNN
+F 2 "" H 5350 7450 50  0001 C CNN
+F 3 "" H 5350 7450 50  0001 C CNN
+	1    5350 7450
 	-1   0    0    -1
 $EndComp
@@
 L power:+5V #PWR0110
 U 1 1 5C55CAF0
-P 5350 6300
-F 0 "#PWR0110" H 5350 6150 50  0001 C CNN
-F 1 "+5V" H 5365 6473 50  0000 C CNN
-F 2 "" H 5350 6300 50  0001 C CNN
-F 3 "" H 5350 6300 50  0001 C CNN
-	1    5350 6300
+P 5350 6550
+F 0 "#PWR0110" H 5350 6400 50  0001 C CNN
+F 1 "+5V" H 5365 6723 50  0000 C CNN
+F 2 "" H 5350 6550 50  0001 C CNN
+F 3 "" H 5350 6550 50  0001 C CNN
+	1    5350 6550
 	-1   0    0    -1
 $EndComp
@@
 L Jumper:Jumper_2_Open JP1
 U 1 1 5C56F029
-P 4150 6750
-F 0 "JP1" H 4150 6985 50  0000 C CNN
-F 1 "Jumper_2_Open" H 4150 6894 50  0000 C CNN
-F 2 "Jumper:SolderJumper-2_P1.3mm_Open_Pad1.0x1.5mm" H 4150 6750 50  0001 C CNN
-F 3 "~" H 4150 6750 50  0001 C CNN
-F 4 "DNP" H 4150 6750 50  0001 C CNN "Variant"
-	1    4150 6750
-	1    0    0    -1
-$EndComp
-Wire Wire Line
-	5400 6550 5350 6550
-Wire Wire Line
-	5350 6550 5350 6300
-Wire Wire Line
-	5350 7200 5350 6950
-Wire Wire Line
-	5350 6950 5400 6950
-Wire Wire Line
-	3000 6750 3000 5500
-Connection ~ 3000 5500
-Wire Wire Line
-	3000 5500 3100 5500
+P 4150 7000
+F 0 "JP1" H 4150 7235 50  0000 C CNN
+F 1 "Jumper_2_Open" H 4150 7144 50  0000 C CNN
+F 2 "Jumper:SolderJumper-2_P1.3mm_Open_Pad1.0x1.5mm" H 4150 7000 50  0001 C CNN
+F 3 "~" H 4150 7000 50  0001 C CNN
+F 4 "DNP" H 4150 7000 50  0001 C CNN "Variant"
+	1    4150 7000
+	1    0    0    -1
+$EndComp
+Wire Wire Line
+	5400 6800 5350 6800
+Wire Wire Line
+	5350 6800 5350 6550
+Wire Wire Line
+	5350 7450 5350 7200
+Wire Wire Line
+	5350 7200 5400 7200
 Wire Wire Line
 	5350 4100 5350 4800
@@
 	4450 5200 5250 5200
 Wire Wire Line
-	4350 6750 4900 6750
+	4350 7000 4900 7000
 Wire Wire Line
 	4900 4600 5500 4600
 Wire Wire Line
-	3000 6750 3950 6750
-Wire Wire Line
-	4900 4600 4900 6750
-Connection ~ 4900 4600
-Connection ~ 4900 6750
-Wire Wire Line
-	4900 6750 5400 6750
-Text Notes 5450 7100 0    50   ~ 0
-Alternativ zum Relay!
+	3000 7000 3950 7000
+Connection ~ 4900 7000
+Wire Wire Line
+	4900 7000 5400 7000
 Wire Wire Line
 	3400 4900 3400 5200
@@
 Wire Wire Line
 	4450 5000 4450 5200
+Wire Notes Line
+	2500 6250 6750 6250
+Wire Wire Line
+	2900 5500 3000 5500
+Wire Wire Line
+	3000 5500 3000 7000
+Connection ~ 3000 5500
+Wire Wire Line
+	3000 5500 3100 5500
+Wire Wire Line
+	4900 4600 4900 7000
+Connection ~ 4900 4600
+Text Notes 5750 6200 0    50   ~ 0
+PLANT
+Text Notes 6250 6375 0    50   ~ 0
+MQTT
+Text Notes 4375 2075 0    50   ~ 0
+use to detect \nwater level
+$Comp
+L Motor:Motor_DC #M?
+U 1 1 5E81B505
+P 6325 4700
+F 0 "#M?" H 6150 4700 50  0001 R CNN
+F 1 "Motor_DC" H 6150 4650 50  0001 R CNN
+F 2 "" H 6325 4610 50  0001 C CNN
+F 3 "~" H 6325 4610 50  0001 C CNN
+F 4 "PLANT" H 6325 4700 50  0001 C CNN "Variant"
+	1    6325 4700
+	1    0    0    -1
+$EndComp
+Wire Notes Line style solid
+	6325 5000 6000 5000
+Wire Notes Line style solid
+	6000 5000 6000 4900
+Wire Notes Line style solid
+	6000 4900 5775 4900
+Wire Notes Line style solid
+	5775 4600 6000 4600
+Wire Notes Line style solid
+	6000 4600 6000 4500
+Wire Notes Line style solid
+	6000 4500 6325 4500
+Wire Notes Line style solid
+	5775 4800 5875 4800
+Wire Notes Line style solid
+	5875 4800 5875 4700
+Wire Notes Line style solid
+	5875 4700 5775 4700
 $EndSCHEMATC

Commit message: kicad-exports and CO2 module
Parts:
- D1, J1, J2, J4, J5, K1, Q3, R1, R2, R3, U4: Variant PIS -> +PIS,-IR
- D2, Q1, R4: Variant PIS, IR -> (none)
- J3, TP1, TP2, TP3, TP4: Variant (none) -> dnp
- JP1, LOGO1, LOGO2: Variant DNP -> dnp
- U1: symbol PIS-rescue:NodeMCU1.0(ESP-12E)-ESP8266 -> ESP8266:NodeMCU_1.0_(ESP-12E)
- U2: Variant IR -> +IR,-PIS
Changed lines of the file:
@@
 Sheet 1 1
 Title "NodeMCU_PIS"
-Date "2020-03-29"
+Date "2020-10-04"
 Rev ""
 Comp "https://nerdyscout.github.io/NodeMCU/PIS"
@@
 F 2 "Symbol:OSHW-Symbol_6.7x6mm_SilkScreen" H 7250 7144 50  0001 C CNN
 F 3 "~" H 7250 6850 50  0001 C CNN
-F 4 "DNP" H 7250 6850 50  0001 C CNN "Variant"
+F 4 "dnp" H 7250 6850 50  0001 C CNN "Variant"
 	1    7250 6850
 	1    0    0    -1
@@
 F 4 "DigiKey" H 3400 2000 50  0001 C CNN "Distributor"
 F 5 "1528-1228-ND" H 3400 2000 50  0001 C CNN "Part Number"
-F 6 "PIS" H 3400 2000 50  0001 C CNN "Variant"
+F 6 "+PIS,-IR" H 3400 2000 50  0001 C CNN "Variant"
 	1    3400 2000
 	-1   0    0    -1
@@
 F 2 "Resistor_THT:R_Axial_DIN0204_L3.6mm_D1.6mm_P7.62mm_Horizontal" V 2930 1550 50  0001 C CNN
 F 3 "~" H 3000 1550 50  0001 C CNN
-F 4 "PIS" H 3000 1550 50  0001 C CNN "Variant"
+F 4 "+PIS,-IR" H 3000 1550 50  0001 C CNN "Variant"
 	1    3000 1550
 	-1   0    0    1
@@
 F 2 "Connector_PinHeader_2.54mm:PinHeader_1x03_P2.54mm_Vertical" H 7800 4750 50  0001 C CNN
 F 3 "~" H 7800 4750 50  0001 C CNN
-F 4 "PIS" H 7800 4750 50  0001 C CNN "Variant"
+F 4 "+PIS,-IR" H 7800 4750 50  0001 C CNN "Variant"
 	1    7800 4750
 	-1   0    0    1
 $EndComp
 $Comp
-L PIS-rescue:NodeMCU1.0(ESP-12E)-ESP8266 U1
+L ESP8266:NodeMCU_1.0_(ESP-12E) U1
 U 1 1 5B936524
 P 8100 2000
@@
 F 2 "Connector_PinHeader_2.54mm:PinHeader_1x04_P2.54mm_Vertical" H 9750 2100 50  0001 C CNN
 F 3 "~" H 9750 2100 50  0001 C CNN
+F 4 "dnp" H 9750 2100 50  0001 C CNN "Variant"
 	1    9750 2100
 	0    1    -1   0
@@
 F 4 "DigiKey" H 3300 5500 50  0001 C CNN "Distributor"
 F 5 "BC547-ND" H 3300 5500 50  0001 C CNN "Part Number"
-F 6 "PIS" H 3300 5500 50  0001 C CNN "Variant"
+F 6 "+PIS,-IR" H 3300 5500 50  0001 C CNN "Variant"
 	1    3300 5500
 	1    0    0    -1
@@
 F 2 "Connector_PinHeader_2.54mm:PinHeader_1x03_P2.54mm_Vertical" H 5050 2000 50  0001 C CNN
 F 3 "~" H 5050 2000 50  0001 C CNN
-F 4 "PIS" H 5050 2000 50  0001 C CNN "Variant"
+F 4 "+PIS,-IR" H 5050 2000 50  0001 C CNN "Variant"
 	1    5050 2000
 	-1   0    0    1
@@
 F 2 "Resistor_THT:R_Axial_DIN0204_L3.6mm_D1.6mm_P7.62mm_Horizontal" V 5680 1600 50  0001 C CNN
 F 3 "~" H 5750 1600 50  0001 C CNN
-F 4 "PIS" H 5750 1600 50  0001 C CNN "Variant"
+F 4 "+PIS,-IR" H 5750 1600 50  0001 C CNN "Variant"
 	1    5750 1600
 	-1   0    0    1
@@
 F 2 "Resistor_THT:R_Axial_DIN0204_L3.6mm_D1.6mm_P7.62mm_Horizontal" V 5680 2400 50  0001 C CNN
 F 3 "~" H 5750 2400 50  0001 C CNN
-F 4 "PIS" H 5750 2400 50  0001 C CNN "Variant"
+F 4 "+PIS,-IR" H 5750 2400 50  0001 C CNN "Variant"
 	1    5750 2400
 	-1   0    0    1
@@
 F 2 "Relay_THT:Relay_SPDT_Omron_G5V-1" H 5280 4670 50  0001 C CNN
 F 3 "http://omronfs.omron.com/en_US/ecb/products/pdf/en-g5v_1.pdf" H 4150 4700 50  0001 C CNN
-F 4 "PIS" H 4150 4700 50  0001 C CNN "Variant"
+F 4 "+PIS,-IR" H 4150 4700 50  0001 C CNN "Variant"
 	1    4150 4700
 	1    0    0    1
@@
 F 2 "Diode_THT:D_DO-35_SOD27_P7.62mm_Horizontal" H 3400 4575 50  0001 C CNN
 F 3 "http://www.nxp.com/documents/data_sheet/1N4148_1N4448.pdf" H 3400 4750 50  0001 C CNN
-F 4 "PIS" H 3400 4750 50  0001 C CNN "Variant"
+F 4 "+PIS,-IR" H 3400 4750 50  0001 C CNN "Variant"
 	1    3400 4750
 	0    -1   1    0
@@
 F 2 "Symbol:KiCad-Logo_6mm_SilkScreen" H 7250 7144 50  0001 C CNN
 F 3 "~" H 7250 6850 50  0001 C CNN
-F 4 "DNP" H 7250 6850 50  0001 C CNN "Variant"
+F 4 "dnp" H 7250 6850 50  0001 C CNN "Variant"
 	1    7250 6850
 	1    0    0    -1
@@
 F 2 "LED_THT:LED_D5.0mm" H 2000 4500 50  0001 C CNN
 F 3 "~" H 2000 4500 50  0001 C CNN
-F 4 "PIS, IR" H 2000 4500 50  0001 C CNN "Variant"
 	1    2000 4500
 	0    -1   -1   0
@@
 F 4 "DigiKey" H 1900 5500 50  0001 C CNN "Distributor"
 F 5 "BC547-ND" H 1900 5500 50  0001 C CNN "Part Number"
-F 6 "PIS, IR" H 1900 5500 50  0001 C CNN "Variant"
 	1    1900 5500
 	1    0    0    -1
@@
 F 2 "TestPoint:TestPoint_Pad_D1.5mm" H 9100 2000 50  0001 C CNN
 F 3 "~" H 9100 2000 50  0001 C CNN
+F 4 "dnp" H 8900 2000 50  0001 C CNN "Variant"
 	1    8900 2000
 	0    1    1    0
@@
 F 2 "TestPoint:TestPoint_Pad_D1.5mm" H 9100 2100 50  0001 C CNN
 F 3 "~" H 9100 2100 50  0001 C CNN
+F 4 "dnp" H 8900 2100 50  0001 C CNN "Variant"
 	1    8900 2100
 	0    1    1    0
@@
 F 2 "TestPoint:TestPoint_Pad_D1.5mm" H 9100 2200 50  0001 C CNN
 F 3 "~" H 9100 2200 50  0001 C CNN
+F 4 "dnp" H 8900 2200 50  0001 C CNN "Variant"
 	1    8900 2200
 	0    1    1    0
@@
 F 2 "TestPoint:TestPoint_Pad_D1.5mm" H 9100 2300 50  0001 C CNN
 F 3 "~" H 9100 2300 50  0001 C CNN
+F 4 "dnp" H 8900 2300 50  0001 C CNN "Variant"
 	1    8900 2300
 	0    1    1    0
@@
 F 2 "Resistor_THT:R_Axial_DIN0204_L3.6mm_D1.6mm_P7.62mm_Horizontal" V 1930 5000 50  0001 C CNN
 F 3 "~" H 2000 5000 50  0001 C CNN
-F 4 "PIS, IR" H 2000 5000 50  0001 C CNN "Variant"
 	1    2000 5000
 	-1   0    0    1
@@
 F 2 "TerminalBlock_TE-Connectivity:TerminalBlock_TE_282834-4_1x04_P2.54mm_Horizontal" H 5700 4800 50  0001 C CNN
 F 3 "~" H 5700 4800 50  0001 C CNN
-F 4 "PIS" H 5700 4800 50  0001 C CNN "Variant"
+F 4 "+PIS,-IR" H 5700 4800 50  0001 C CNN "Variant"
 	1    5700 4800
 	1    0    0    1
@@
 F 2 "Connector_PinHeader_2.54mm:PinHeader_1x04_P2.54mm_Vertical" H 9300 4850 50  0001 C CNN
 F 3 "~" H 9300 4850 50  0001 C CNN
-F 4 "PIS" H 9300 4850 50  0001 C CNN "Variant"
+F 4 "+PIS,-IR" H 9300 4850 50  0001 C CNN "Variant"
 	1    9300 4850
 	-1   0    0    1
@@
 F 2 "OptoDevice:Vishay_CAST-3Pin" H 5750 6625 50  0001 C CNN
 F 3 "http://www.micropik.com/PDF/tsop17xx.pdf" H 6450 7300 50  0001 C CNN
-F 4 "IR" H 5800 7000 50  0001 C CNN "Variant"
+F 4 "+IR,-PIS" H 5800 7000 50  0001 C CNN "Variant"
 	1    5800 7000
 	-1   0    0    -1
@@
 F 2 "Jumper:SolderJumper-2_P1.3mm_Open_Pad1.0x1.5mm" H 4150 7000 50  0001 C CNN
 F 3 "~" H 4150 7000 50  0001 C CNN
-F 4 "DNP" H 4150 7000 50  0001 C CNN "Variant"
+F 4 "dnp" H 4150 7000 50  0001 C CNN "Variant"
 	1    4150 7000
 	1    0    0    -1
@@
 use to detect \nwater level
 $Comp
-L Motor:Motor_DC #M?
+L Motor:Motor_DC #M1
 U 1 1 5E81B505
 P 6325 4700
-F 0 "#M?" H 6150 4700 50  0001 R CNN
+F 0 "#M1" H 6150 4700 50  0001 R CNN
 F 1 "Motor_DC" H 6150 4650 50  0001 R CNN
 F 2 "" H 6325 4610 50  0001 C CNN
