File: PWR/PWR.sch (KiCad schematic (older format))
At the start: 19 parts, among them J1 Screw_Terminal_01x04, J2 Conn_01x01, J3 Conn_01x02, J5 Conn_01x01, Q1 TIC206, U1 MOC3021M, U2 4N25, U3 NodeMCU1.0(ESP-12E)

Commit message: kicad-exports and CO2 module
Parts:
- PS1: symbol PWR-rescue:IRM-02-5-Converter_ACDC-Power-rescue-PWR-rescue -> Converter_ACDC:IRM-02-5
- U1: symbol PWR-rescue:MOC3021M-Relay_SolidState-Power-rescue-PWR-rescue -> Relay_SolidState:MOC3021M
- U3: symbol PWR-rescue:NodeMCU1.0(ESP-12E)-ESP8266-Power-rescue-PWR-rescue -> ESP8266:NodeMCU_1.0_(ESP-12E)
Changed lines of the file:
@@
 Sheet 1 1
 Title "NodeMCU_PWR"
-Date "2020-03-29"
+Date "2020-10-04"
 Rev ""
 Comp "https://nerdyscout.github.io/NodeMCU/PWR"
@@
 $EndComp
 $Comp
-L PWR-rescue:MOC3021M-Relay_SolidState-Power-rescue-PWR-rescue U1
+L Relay_SolidState:MOC3021M U1
 U 1 1 5B9C0A53
 P 3900 5500
@@
 	1750 2700 1900 2700
 $Comp
-L PWR-rescue:IRM-02-5-Converter_ACDC-Power-rescue-PWR-rescue PS1
+L Converter_ACDC:IRM-02-5 PS1
 U 1 1 5B9C1D83
 P 6750 2000
@@
 $EndComp
 $Comp
-L PWR-rescue:NodeMCU1.0(ESP-12E)-ESP8266-Power-rescue-PWR-rescue U3
+L ESP8266:NodeMCU_1.0_(ESP-12E) U3
 U 1 1 5B6B53D8
 P 2700 2100
